File: docs/KiCad/MorayGlow.kicad_sch (KiCad schematic)
At the start: 24 parts, among them J2 RGB LED, J5 Barrel Jack, Q1 IRLML6344TRPBF, Q2 IRLML6344TRPBF, Q3 IRLML6344TRPBF, SW1 SW_DIP_x01, U1 XIAO-ESP32-S3-Plus-SMD

Commit message: Apply schematic review changes: GPIO fix, component updates, new KiCad files
- Fix critical bug: PIN_BLUE moved from GPIO3 to GPIO6 (D5) — GPIO3 is an
  ESP32-S3 strapping pin that could cause boot issues
- R4/R5/R6 gate pull-downs changed 10kΩ → 100kΩ (saves ~1mA, adequate for
  IRLML6344 gate leakage)
- C3 moved from VCC_12V input to VDD_5V output of MP1584 (correct placement)
- C4 100µF added on VCC_12V at J2 to absorb PWM switching transients
- Update KiCad schematic, PCB, and project files with all reviewed changes
- Update docs/Hardware/BOM.csv, circuit_reference.txt, and docs/index.html
- Remove stale fabrication-toolkit production outputs (can be regenerated)
- Add KiCad .lck files to .gitignore

Co-Authored-By: Claude Sonnet 4.6 <noreply@anthropic.com>
Parts:
- added C4: 100uF, Capacitor_Tantalum_SMD:CP_EIA-3216-18_Kemet-A, symbol Device:C_Polarized_Small
- J2: footprint Connector_JST:JST_SH_SM04B-SRSS-TB_1x04-1MP_P1.00mm_Horizontal -> Connector_JST:JST_XH_S4B-XH-A_1x04_P2.50mm_Horizontal
- Q1: renamed from Q3; footprint Package_TO_SOT_SMD:SOT-23 -> IRLML6344TRPBF:TRANS_IRLML6344TRPBF
- Q2: renamed from Q1; footprint Package_TO_SOT_SMD:SOT-23 -> IRLML6344TRPBF:TRANS_IRLML6344TRPBF
- Q3: renamed from Q2; footprint Package_TO_SOT_SMD:SOT-23 -> IRLML6344TRPBF:TRANS_IRLML6344TRPBF
- R4: renamed from R6; value 10k -> 100k
- R5: renamed from R4; value 10k -> 100k
- R6: renamed from R5; value 10k -> 100k
- renumbered J5 to J1, R3 to R1, R1 to R2, R2 to R3
Connections:
- net RGB_B: now also U1.6 (GPIO6_A5_D5_SCL); no longer U1.3 (GPIO3_A2_D2)
- net VCC_12V: now also C4.1; no longer C3.1
- net VDD_5V: now also C3.2
- net GND: now reaches PS1.2 (Pin_2)
- net GND: now also C1.2, C2.2, C3.1, H1.1, H2.1, H3.1, H4.1, J1.3, LED1.1 (K), PS1.4 (Pin_4), Q1.2, Q2.2, Q3.2, R4.2, R5.2, R6.2, SW1.2, U1.13 (GND), U1.27 (GND1), U1.33 (GND2), U1.34 (PAD), C4.2
- no-connect marks 4 -> 26
Other:
- moved on the sheet: C3, J2, PS1, Q1, Q2, Q3, R1, R2, R3, R4, R5, R6
